File: buffered-mult/pcb/buffered-mult.brd (EAGLE design)
At the start: 100 x 15 mm, 34 parts, among them J1 WQP_PJ_301BM, J2 WQP_PJ_301BM, J3 WQP_PJ_301BM, J4 WQP_PJ_301BM, J5 WQP_PJ_301BM, J6 WQP_PJ_301BM, J7 WQP_PJ_301BM, J8 WQP_PJ_301BM, U1 TL072_SMD, U2 TL072_SMD

Commit message: previous attempt - won't work
Parts:
- added C7, C8: (no value), rcl:PANASONIC_D
- added D1, D2: (no value), diode:SOD123
- J1, J2, J3, J4, J5, J6, J7, J8: device mjb-pots:WQP_PJ_301BM -> mjb-parts:WQP_PJ_301BM
- moved R17 14.7 mm to (57.3, 7.40), turned to 90 degrees
- moved R11 14.5 mm to (61.5, 7.40), turned to 90 degrees
- moved C5 10.4 mm to (70.2, 7.40), turned to 270 degrees
- moved C6 9.63 mm to (59.4, 7.40), turned to 90 degrees
- moved C1 9.30 mm to (55.9, 4.10)
- moved R14 8.20 mm to (57.2, 10.9)
- moved C3 7.93 mm to (94.6, 5.90), turned to 180 degrees
- moved R13 7.63 mm to (72.3, 7.40), turned to 90 degrees
- moved R10 6.60 mm to (74.9, 11.5), turned to 270 degrees
- moved R16 6.32 mm to (71.7, 10.0)
- moved R15 4.97 mm to (80.3, 7.30), turned to 90 degrees
- moved C4 4.88 mm to (82.4, 7.30), turned to 90 degrees
- moved R3 4.41 mm to (83.0, 4.70), turned to 180 degrees
- moved R4 3.99 mm to (71.7, 4.80), turned to 180 degrees
- moved R12 3.94 mm to (79.7, 10.8), turned to 0 degrees
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Connections:
- new net N$10: SV1.10, SV1.9
- new net N$11: SV1.1, SV1.2
- net GND: now also C7.-, C8.+, D1.A, D2.C
- net VCC: now also C7.+, D1.C; no longer SV1.10, SV1.9
- net VEE: now also C8.-, D2.A; no longer SV1.1, SV1.2
Routing:
- net GND: track 0.00 -> 129.5 mm, vias 0 -> 2
- net VCC: track 0.00 -> 76.7 mm, vias 0 -> 1
- net N$16: track 0.00 -> 54.7 mm
- net VEE: track 0.00 -> 54.1 mm, vias 0 -> 2
- net N$22: track 0.00 -> 20.6 mm
- net N$3: track 0.00 -> 16.4 mm, vias 0 -> 2
- net N$9: track 0.00 -> 14.9 mm
- net N$2: track 0.00 -> 13.3 mm
- net N$20: track 0.00 -> 11.5 mm, vias 0 -> 1
- net N$7: track 0.00 -> 11.0 mm
- net N$14: track 0.00 -> 11.0 mm
- net N$13: track 0.00 -> 9.61 mm
- net N$4: track 0.00 -> 8.34 mm
- net N$19: track 0.00 -> 7.44 mm
- net N$15: track 0.00 -> 7.05 mm
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Other:
- board size 100 x 15 mm -> 100 x 15.5 mm
