File: buffered-mult/pcb/buffered-mult.sch (EAGLE design)
At the start: 34 parts, among them J1 WQP_PJ_301BM, J2 WQP_PJ_301BM, J3 WQP_PJ_301BM, J4 WQP_PJ_301BM, J5 WQP_PJ_301BM, J6 WQP_PJ_301BM, J7 WQP_PJ_301BM, J8 WQP_PJ_301BM, U1 TL072_SMD, U2 TL072_SMD

Commit message: previous attempt - won't work
Parts:
- added C7, C8: (no value), rcl:CPOL-USD
- added D1, D2: (no value), diode:DIODE-SOD123
- J1, J2, J3, J4, J5, J6, J7, J8: device mjb-pots:WQP_PJ_301BM -> mjb-parts:WQP_PJ_301BM
Connections:
- new net N$10: SV1.10, SV1.9
- new net N$11: SV1.1, SV1.2
- net GND: now also C7.-, C8.+, D1.A, D2.C
- net VCC: now also C7.+, D1.C; no longer SV1.10, SV1.9
- net VEE: now also C8.-, D2.A; no longer SV1.1, SV1.2
Other:
- moved on the sheet: C1
